File: PCB_Sender/PCB_Sender.kicad_sch (KiCad schematic)
At the start: 29 parts, among them J1 Power-Pass_MCU, J2 Header A, J3 NTC_0-3, J4 NTC_Internal, J5 Power-Pass_PSU, J7 Header B, SW1 SW_Wuerth_450301014042, U1 ESP32-DEVKITC-32D, U2 TP4056 Module, U3 DC/DC Module

Commit message: WiP commit
Commited work in progress
Parts:
- removed C1: 10V, 220uF, Capacitor_THT:CP_Radial_D6.3mm_P2.50mm, symbol Device:C_Polarized
- removed H1, H2, H3, H4: MountingHole, MountingHole:MountingHole_3.2mm_M3_DIN965, symbol Mechanical:MountingHole
- removed J1: Power-Pass_MCU, Connector_Molex:Molex_Mini-Fit_Jr_5569-04A2_2x02_P4.20mm_Horizontal, symbol Connector_Generic:Conn_02x02_Top_Bottom
- removed J3: NTC_0-3, TerminalBlock_TE-Connectivity:TerminalBlock_TE_282834-8_1x08_P2.54mm_Horizontal, symbol Connector:Screw_Terminal_01x08
- removed J5: Power-Pass_PSU, Connector_Molex:Molex_Mini-Fit_Jr_5569-04A2_2x02_P4.20mm_Horizontal, symbol Connector_Generic:Conn_02x02_Top_Bottom
- added C1, C5: 50V, 100nF, Capacitor_SMD:C_1206_3216Metric, symbol Device:C
- added C6: 10V, 220uF, Capacitor_THT:CP_Radial_D6.3mm_P2.50mm, symbol Device:C_Polarized
- added G1: AUGA-Tech-LOGO, 0_user_lib:AUGA-Tech-footprint, symbol 0_user_lib:AUGA-Tech-LOGO
- added J6: DTM13-12PA, 0_user_lib:DTM13-12PA-R008, symbol 0_user_lib:DTM13-12PA-R008
- added R12, R9: 100K, Resistor_SMD:R_0805_2012Metric, symbol Device:R_Small
- added U4: LM7805_TO220, Package_TO_SOT_SMD:TO-252-2, symbol Regulator_Linear:LM7805_TO220
- C2, C4: value 100nF -> 50V, 100nF; footprint Capacitor_THT:C_Disc_D3.8mm_W2.6mm_P2.50mm -> Capacitor_SMD:C_1206_3216Metric; JLCPCB Part # (none) -> C24497; Package (none) -> 1206
- C3: Part No 860020273009 -> (none)
- D1: now not fitted
- D2: footprint LED_THT:LED_D5.0mm -> LED_SMD:LED_0805_2012Metric; JLCPCB Part # (none) -> C2297; Package (none) -> 0805
- R1, R2, R3, R4, R5: footprint Resistor_THT:R_Axial_DIN0207_L6.3mm_D2.5mm_P10.16mm_Horizontal -> Resistor_SMD:R_0805_2012Metric; JLCPCB Part # (none) -> C17414; Package (none) -> 0805
- R6, R7: footprint Resistor_THT:R_Axial_DIN0207_L6.3mm_D2.5mm_P10.16mm_Horizontal -> Resistor_SMD:R_0805_2012Metric; JLCPCB Part # (none) -> C149504; Package (none) -> 0805
- R8: value 560 -> 680; footprint Resistor_THT:R_Axial_DIN0207_L6.3mm_D2.5mm_P10.16mm_Horizontal -> Resistor_SMD:R_0805_2012Metric; JLCPCB Part # (none) -> C17798; Package (none) -> 0805
- SW1: value SW_Wuerth_450301014042 -> On-Off Switch; footprint Button_Switch_THT:SW_Slide-03_Wuerth-WS-SLTV_10x2.5x6.4_P2.54mm -> Button_Switch_THT:SW_Slide_SPDT_Straight_CK_OS102011MS2Q; MFR (none) -> C&K; MPN (none) -> OS102011MS2QS1
- U1: footprint local_lib:MODULE_ESP32-DEVKITC-32D -> 0_user_lib:MODULE_ESP32-DEVKITC-32D; MF Espressif Systems -> (none)
- U2: footprint local_lib:TP4056-Module -> 0_user_lib:TP4056-Module
- U3: footprint local_lib:DCDC_StepUp -> 0_user_lib:DCDC_StepUp
Connections:
- net BAT- is gone; now on net GND: BT1.2 (-), U2.6 (B-)
- net GND1 is gone; now on net GND: J7.6 (Pin_6), U1.J2-14 (GND1)
- net PSU_5V is gone; now on net +5V: C3.1, C4.1, R8.2, U3.3 (Vout)
- net PSU_GND is gone; now on net GND: C3.2, C4.2, D2.1 (K), U3.4 (GND)
- net +3V3: now also J6.10, J6.7, J6.8, J6.9, R12.2, R9.2
- net +5V: no longer C2.1
- net GND: now also U2.2 (CHG-), U2.4 (OUT-), U3.2 (GND), C1.2, C5.2, C6.2, J6.12, J6.13 (GND), J6.2, U4.2 (GND)
- net NTC_0: now also J6.3
- net NTC_1: now also J6.4
- net NTC_2: now also J6.5
- net NTC_3: now also J6.6
- net VCC: now also C1.1, C5.1, J6.1, U4.1 (VI); no longer R6.2
- net +5C: now reaches U2.1 (CHG+)
- net +5C: now also C2.1, C6.1, U4.3 (VO)
- net BAT+ renamed +BATT
- net +BATT: now also R6.2
- net IO12 renamed Wheel_Side
- net Wheel_Side: now also J6.11, R12.1, R9.1
- no-connect marks 4 -> 2
Other:
- note added: "4.8mA @ 5V"
- note added: "Adressable RGB LED (Optional)"
- note added: "If Wheel Side pin is pulled to GND, Then it is Right Side wheel. If left floating - Left Side"
- note added: "It should be charged from 12-24v 1st option: Lemona DC/DC su LM2596S Įėjimas 3-40VDC iki 2A 2nd option: LM7805"
- note added: "Vin 7v-35V"
- note added: "Wheel side pin pull-up"
- note removed: "Jungtis, perduoti 5V ir Baterijos Įtampą Į pagrindinį vadliklį"
- note removed: "NTC probe connection points"
- note removed: "Power passthrough connectors are needed to be able to disconnect battery module for recharging / replacement. Without disconnecting the whole MCU module. Because MCU module will have NTC sensors glued to the wheel."
- moved on the sheet: C2, R1, R2, R3, R4, R5

Commit message: PCB updates
Other:
- note added: "Need Heatsink !"
- note added: "REV D requirements: Power led is too bright Add Status LED to IO21 pin routing fix, from battery + RUN DRC!!! LM7805 needs heatsink, more space for it. Add Reverse voltage protection More el. caps for all busses"
- note removed: "It should be charged from 12-24v 1st option: Lemona DC/DC su LM2596S Įėjimas 3-40VDC iki 2A 2nd option: LM7805"
Changed lines of the file:
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@@
 		)
 	)
-	(text "It should be charged from 12-24v\n\n1st option: Lemona DC/DC su LM2596S Įėjimas 3-40VDC iki 2A\n\n2nd option: LM7805"
+	(text "REV D requirements:\nPower led is too bright\nAdd Status LED to IO21 pin\nrouting fix, from battery +\nRUN DRC!!!\nLM7805 needs heatsink, more space for it. Add Reverse voltage protection\nMore el. caps for all busses"
 		(exclude_from_sim no)
-		(at 18.034 23.368 0)
+		(at 13.97 21.59 0)
 		(effects
 			(font
 				(size 1.27 1.27)
+				(thickness 0.254)
+				(bold yes)
 			)
 			(justify left)
@@
 		)
 	)
+	(text "Need Heatsink !"
+		(exclude_from_sim no)
+		(at 71.882 39.878 0)
+		(effects
+			(font
+				(size 1.27 1.27)
+			)
+		)
+	)
