File: HV_BAT_COM_Distribution_Board/HV_BAT_COM_Distribution_Board.kicad_pcb (KiCad board)
At the start: 2 copper layers, 110 x 91 mm, 36 parts, among them J1 CAN1, J10 T2, J11 T3, J12 T4, J13 HVIL 1, J14 USB_B, J15 T5, J16 USB, J17 Pre-Charge, J18 HVIL 2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

Commit message: PCB updates
Parts:
- added D10: FB2 (Green), LED_SMD:LED_0805_2012Metric, F.Cu at (160.0, 97.5)
- added D11: Power OK (Red), LED_SMD:LED_0805_2012Metric, F.Cu at (167.5, 97.5)
- added D12: FB2 (Green), LED_SMD:LED_0805_2012Metric, F.Cu at (165.0, 97.5)
- added D7: Precharge (Green), LED_SMD:LED_0805_2012Metric, F.Cu at (162.5, 97.5)
- added D8: IGN (Yellow), LED_SMD:LED_0805_2012Metric, F.Cu at (170.0, 97.5)
- added D9: FB1 (Green), LED_SMD:LED_0805_2012Metric, F.Cu at (157.5, 97.5)
- added G1: AUGA-Tech-LOGO, 0_user_lib:AUGA-Tech-LOGO_12x15, B.Cu at (152.7, 103.0)
- added R10: 1k5, Resistor_SMD:R_0805_2012Metric, F.Cu at (165.0, 94.0)
- added R5: 1k5, Resistor_SMD:R_0805_2012Metric, F.Cu at (162.5, 94.0)
- added R6: 1k5, Resistor_SMD:R_0805_2012Metric, F.Cu at (157.5, 94.0)
- added R7: 1k5, Resistor_SMD:R_0805_2012Metric, F.Cu at (170.0, 94.0)
- added R8: 1k5, Resistor_SMD:R_0805_2012Metric, F.Cu at (160.0, 94.0)
- added R9: 1k5, Resistor_SMD:R_0805_2012Metric, F.Cu at (167.5, 94.0)
- added SW2: SW_DIP_x01, Button_Switch_THT:SW_DIP_SPSTx01_Slide_9.78x4.72mm_W7.62mm_P2.54mm, F.Cu at (139.9, 131.4)
- D6: value Power OK -> Power OK (Red)
- G1: footprint 0_user_lib:AUGA-Tech-footprint -> 0_user_lib:AUGA-Tech-LOGO_12x15
- J14: footprint Connector_USB:USB_B_Lumberg_2411_02_Horizontal -> Connector_USB:USB_B_TE_5787834_Vertical
- SW1: footprint Button_Switch_SMD:SW_DIP_SPSTx01_Slide_9.78x4.72mm_W8.61mm_P2.54mm -> Button_Switch_THT:SW_DIP_SPSTx01_Slide_9.78x4.72mm_W7.62mm_P2.54mm
- moved R4 96.6 mm to (172.5, 94.0), turned to -90 degrees
- moved D6 94.2 mm to (172.5, 97.5), turned to 90 degrees
- moved G1 70.1 mm to (100.0, 77.3), turned to 90 degrees
- moved SW1 4.61 mm to (184.3, 109.1), turned to 180 degrees
- moved J14 4.03 mm to (119.8, 133.9)
- moved R1 2.87 mm to (144.5, 139.4), turned to 0 degrees
Connections:
- J2 pad 14: unconnected-(J2-Pin_14-Pad14) -> /ERROR
- J2 pad 15: unconnected-(J2-Pin_15-Pad15) -> /READY
- J6 pad 22: unconnected-(J6-Pin_22-Pad22) -> GND
- J6 pad 3: unconnected-(J6-Pin_3-Pad3) -> /CAN_1H
- J6 pad 4: unconnected-(J6-Pin_4-Pad4) -> /CAN_1L
- J6 pad 6: unconnected-(J6-Pin_6-Pad6) -> /CAN_2H
- J6 pad 7: unconnected-(J6-Pin_7-Pad7) -> /CAN_2L
- R1 pad 1: /CAN_1H -> Net-(R1-Pad1)
Routing:
- net +12V: track 0.00 -> 277.6 mm, vias 0 -> 2
- net /CAN_1L: track 0.00 -> 208.9 mm, vias 0 -> 3
- net /CAN_1H: track 0.00 -> 197.4 mm, vias 0 -> 3
- net /CAN_2H: track 0.00 -> 197.4 mm, vias 0 -> 2
- net /CAN_2L: track 0.00 -> 169.9 mm, vias 0 -> 1
- net /HVIL_OUT: track 0.00 -> 120.9 mm
- net /HVIL_IN: track 0.00 -> 119.2 mm, vias 0 -> 2
- net /CONT_PWR: track 0.00 -> 99.1 mm, vias 0 -> 2
- net /PRECHARGE: track 0.00 -> 96.6 mm, vias 0 -> 1
- net /POS_FB: track 0.00 -> 95.7 mm, vias 0 -> 3
- net /CONT: track 0.00 -> 89.9 mm, vias 0 -> 1
- net /NEG_FB: track 0.00 -> 89.2 mm, vias 0 -> 2
- net Net-(J7-Pin_19): track 0.00 -> 74.5 mm
- net /POS_CONT: track 0.00 -> 72.0 mm, vias 0 -> 1
- net /HV_FB: track 0.00 -> 71.5 mm
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Other:
- board text added: "CAN-1 Terminator"
- board text added: "D. Vaitiekus 2024-06-17 HV-BAT-COM REV A AUGA Tech"
- board text added: "ERROR"
- board text added: "FB1"
- board text added: "FB2"
- board text added: "H"
- board text added: "IGN"
- board text added: "L"
- board text added: "PRCHRG"
- board text added: "PWR_OK"
- board text added: "READY"
- board text removed: "CAN-1"
- board text removed: "CAN-1 120R"
- board text removed: "OFF"
- board text removed: "ON"
