File: HV_BAT_COM_Distribution_Board/HV_BAT_COM_Distribution_Board.kicad_sch (KiCad schematic)
At the start: 36 parts, among them J1 CAN1, J10 T2, J11 T3, J12 T4, J13 HVIL 1, J14 USB_B, J15 T5, J16 USB, J17 Pre-Charge, J18 HVIL 2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

Commit message: PCB updates
Parts:
- added D10, D12: FB2 (Green), LED_SMD:LED_0805_2012Metric, symbol Device:LED
- added D11: Power OK (Red), LED_SMD:LED_0805_2012Metric, symbol Device:LED
- added D7: Precharge (Green), LED_SMD:LED_0805_2012Metric, symbol Device:LED
- added D8: IGN (Yellow), LED_SMD:LED_0805_2012Metric, symbol Device:LED
- added D9: FB1 (Green), LED_SMD:LED_0805_2012Metric, symbol Device:LED
- added R10, R5, R6, R7, R8, R9: 1k5, Resistor_SMD:R_0805_2012Metric, symbol Device:R
- added SW2: SW_DIP_x01, Button_Switch_THT:SW_DIP_SPSTx01_Slide_9.78x4.72mm_W7.62mm_P2.54mm, symbol Switch:SW_DIP_x01
- D6: value Power OK -> Power OK (Red)
- G1: footprint 0_user_lib:AUGA-Tech-footprint -> 0_user_lib:AUGA-Tech-LOGO_12x15; now not fitted
- H1, H2, H3, H4: now not fitted
- J1, J16, J4, J5, J8: Package Plugin,P=3mm -> Plugin,P=3mm
- J10, J11, J12, J13, J15, J17, J18, J9: JLCPCB Part # (none) -> C293362; Package (none) -> Plugin,P=3mm
- J14: footprint Connector_USB:USB_B_Lumberg_2411_02_Horizontal -> Connector_USB:USB_B_TE_5787834_Vertical; JLCPCB Part # (none) -> C592900; MPN 61400416121 -> 61400413321; Package (none) -> Plugin
- J2, J3, J6, J7: JLCPCB Part # (none) -> C492366; Package (none) -> Plugin,P=3mm
- K1, K2: JLCPCB Part # (none) -> C225715; Package (none) -> Plugin,10x20mm
- SW1: footprint Button_Switch_SMD:SW_DIP_SPSTx01_Slide_9.78x4.72mm_W8.61mm_P2.54mm -> Button_Switch_THT:SW_DIP_SPSTx01_Slide_9.78x4.72mm_W7.62mm_P2.54mm; JLCPCB Part # (none) -> C126888; Package (none) -> Plugin,9.9x4mm
Connections:
- net CAN_1H: now also J6.3 (Pin_3), SW2.1; no longer R1.1
- net CAN_1L: now also J6.4 (Pin_4)
- net CAN_2H: now also J6.6 (Pin_6)
- net CAN_2L: now also J6.7 (Pin_7)
- net GND: now also J6.22 (Pin_22), D10.1 (K), D11.1 (K), D12.1 (K), D7.1 (K), D8.1 (K), D9.1 (K)
- net IGN: now also R7.1
- net NEG_FB: now also R8.1
- net POS_FB: now also R6.1
- net PRECHARGE: now also R5.1
- net ERROR: now reaches J2.14 (Pin_14)
- net ERROR: now also R9.1
- net READY: now reaches J2.15 (Pin_15)
- net READY: now also R10.1
- new net: R1.1, SW2.2
- new net: D8.2 (A), R7.2
- new net: D11.2 (A), R9.2
- new net: D12.2 (A), R10.2
- new net: D9.2 (A), R6.2
- new net: D10.2 (A), R8.2
- new net: D7.2 (A), R5.2
- no-connect marks 32 -> 42
Other:
- note added: "Optional CAN1 120 Ohm Terminator"
- note added: "Vertical USB Type B"
- note removed: "CAN1 Line Terminator"
- moved on the sheet: D1, D2, D3, D4, D5, D6, J4, J5, K1, R1, R4
