File: PCB_Receiver/PCB_Receiver.kicad_pcb (KiCad board)
At the start: 2 copper layers, 53 x 99 mm, 20 parts, among them J1 MCP-2515-CAN, J2 CAN_passthrough, J3 Power Input 12V, J6 Header A, J8 Header B, SW2 Switch, U4 ESP32-WROOM-32UE, U5 DC StepDown

Commit message: PCB updates
Routing:
- net +5V: track 136.2 -> 139.2 mm
Changed lines of the file:
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@@
 		)
 		(property "Value" "CAN_passthrough"
-			(at 0 4.87 360)
+			(at 0 4.87 0)
 			(layer "F.Fab")
 			(effects
@@
 	)
 	(segment
+		(start 154 92.25)
+		(end 153.75 92)
+		(width 0.5)
+		(layer "F.Cu")
+		(net 3)
+	)
+	(segment
 		(start 161.5 116)
 		(end 152 106.5)
@@
 		(width 0.5)
 		(layer "F.Cu")
+		(net 3)
+	)
+	(segment
+		(start 154 94.92)
+		(end 154 92.25)
+		(width 0.5)
+		(layer "F.Cu")
