File: Temperature_cluster/CANBUS.kicad_sch (KiCad schematic)
At the start: 13 parts, among them U8 TJA1051T-3

Commit message: PCB updates
Parts:
- added TP6: CANH, TestPoint:TestPoint_THTPad_D1.0mm_Drill0.5mm, symbol Connector:TestPoint
- added TP7: CANL, TestPoint:TestPoint_THTPad_D1.0mm_Drill0.5mm, symbol Connector:TestPoint
- C33: JLCPCB Part # (none) -> C565636; Package (none) -> 0805
Connections:
- net CAN_H: now also TP6.1
- net CAN_L: now also TP7.1
Other:
- company: AUGA Tech -> D. Vaitiekus
Changed lines of the file:
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@@
 	(title_block
 		(title "CAN-Transceiver")
-		(date "2024-05-28")
+		(date "2024-06-28")
 		(rev "A")
-		(company "AUGA Tech")
-		(comment 1 "Darius Vaitiekus")
+		(company "D. Vaitiekus")
+		(comment 1 "AUGA Tech")
+	)
+	(junction
+		(at 219.71 55.88)
+		(diameter 0)
+		(color 0 0 0 0)
 	)
 	(junction
@@
 	)
 	(junction
+		(at 219.71 43.18)
+		(diameter 0)
+		(color 0 0 0 0)
+	)
+	(junction
 		(at 127 36.83)
 		(diameter 0)
@@
 	(wire
 		(pts
+			(xy 219.71 43.18) (xy 223.52 43.18)
+		)
+		(stroke
+			(width 0)
+			(type default)
+		)
+	)
+	(wire
+		(pts
 			(xy 146.05 34.29) (xy 146.05 36.83)
 		)
@@
 	(wire
 		(pts
-			(xy 210.82 43.18) (xy 223.52 43.18)
+			(xy 210.82 43.18) (xy 219.71 43.18)
 		)
 		(stroke
@@
 	(wire
 		(pts
+			(xy 219.71 55.88) (xy 223.52 55.88)
+		)
+		(stroke
+			(width 0)
+			(type default)
+		)
+	)
+	(wire
+		(pts
 			(xy 87.63 54.61) (xy 96.52 54.61)
 		)
@@
 	(wire
 		(pts
-			(xy 210.82 55.88) (xy 223.52 55.88)
+			(xy 210.82 55.88) (xy 219.71 55.88)
 		)
 		(stroke
@@
 			)
 		)
+		(property "JLCPCB Part #" "C565636"
+			(at 240.03 49.53 0)
+			(effects
+				(font
+					(size 1.27 1.27)
+				)
+				(hide yes)
+			)
+		)
+		(property "Package" "0805"
+			(at 240.03 49.53 0)
+			(effects
+				(font
+					(size 1.27 1.27)
+				)
+				(hide yes)
+			)
+		)
 		(pin "2"
 		)
@@
 	)
 	(symbol
+		(lib_id "Connector:TestPoint")
+		(at 219.71 43.18 0)
+		(unit 1)
+		(exclude_from_sim no)
+		(in_bom yes)
+		(on_board yes)
+		(dnp no)
+		(fields_autoplaced yes)
+		(property "Reference" "TP6"
+			(at 222.25 38.6079 0)
+			(effects
+				(font
+					(size 1.27 1.27)
+				)
+				(justify left)
+			)
+		)
+		(property "Value" "CANH"
+			(at 222.25 41.1479 0)
+			(effects
+				(font
+					(size 1.27 1.27)
+				)
+				(justify left)
+			)
+		)
+		(property "Footprint" "TestPoint:TestPoint_THTPad_D1.0mm_Drill0.5mm"
+			(at 224.79 43.18 0)
+			(effects
+				(font
+					(size 1.27 1.27)
+				)
+				(hide yes)
+			)
+		)
+		(property "Datasheet" "~"
+			(at 224.79 43.18 0)
+			(effects
+				(font
+					(size 1.27 1.27)
+				)
+				(hide yes)
+			)
+		)
+		(property "Description" "test point"
+			(at 219.71 43.18 0)
+			(effects
+				(font
+					(size 1.27 1.27)
+				)
+				(hide yes)
+			)
+		)
+		(pin "1"
+		)
+		(instances
+			(project "Temperature_cluster"
+				(path "/c96faf72-0ed2-4ed1-a439-4e57053e11b5/6bce3d65-0be4-4e8d-bb75-91c3cf81a4ae"
+					(reference "TP6")
+					(unit 1)
+				)
+			)
+		)
+	)
+	(symbol
 		(lib_id "Device:C_Polarized_Small")
 		(at 114.3 33.02 90)
@@
 					(unit 1)
 				)
+			)
+		)
+	)
+	(symbol
+		(lib_id "Connector:TestPoint")
+		(at 219.71 55.88 180)
+		(unit 1)
+		(exclude_from_sim no)
+		(in_bom yes)
+		(on_board yes)
+		(dnp no)
+		(fields_autoplaced yes)
+		(property "Reference" "TP7"
+			(at 222.25 57.9119 0)
+			(effects
+				(font
+					(size 1.27 1.27)
+				)
+				(justify right)
+			)
+		)
+		(property "Value" "CANL"
+			(at 222.25 60.4519 0)
+			(effects
+				(font
+					(size 1.27 1.27)
+				)
+				(justify right)
+			)
+		)
+		(property "Footprint" "TestPoint:TestPoint_THTPad_D1.0mm_Drill0.5mm"
+			(at 214.63 55.88 0)
+			(effects
+				(font
+					(size 1.27 1.27)
+				)
+				(hide yes)
+			)
+		)
+		(property "Datasheet" "~"
+			(at 214.63 55.88 0)
+			(effects
+				(font
+					(size 1.27 1.27)
+				)
+				(hide yes)
+			)
+		)
+		(property "Description" "test point"
+			(at 219.71 55.88 0)
+			(effects
+				(font
+					(size 1.27 1.27)
+				)
+				(hide yes)
+			)
+		)
+		(pin "1"
+		)
+		(instances
+			(project "Temperature_cluster"
+				(path "/c96faf72-0ed2-4ed1-a439-4e57053e11b5/6bce3d65-0be4-4e8d-bb75-91c3cf81a4ae"
+					(reference "TP7")
+					(unit 1)
+				)
