File: Temperature_cluster/PSU.kicad_sch (KiCad schematic)
At the start: 37 parts, among them U6 TPS5430DDAR, U7 AMS1117-3.3

Commit message: PCB updates
Parts:
- added TP5: 3v3, TestPoint:TestPoint_THTPad_D1.0mm_Drill0.5mm, symbol Connector:TestPoint
- L2: JLCPCB Part # C216156 -> C171763; Package L0805 -> 1206
Connections:
- net +3V3: now also TP5.1
Other:
- note added: "Input range 14V-36V"
- company: (none) -> D. Vaitiekus
- title: (none) -> Power Module
Changed lines of the file:
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@@
 	(generator_version "8.0")
 	(paper "A4")
+	(title_block
+		(title "Power Module")
+		(date "2024-06-28")
+		(rev "A")
+		(company "D. Vaitiekus")
+		(comment 1 "AUGA Tech")
+	)
 	(junction
 		(at 67.31 92.71)
@@
 		)
 	)
+	(text "Input range\n14V-36V"
+		(exclude_from_sim no)
+		(at 37.592 40.386 0)
+		(effects
+			(font
+				(size 1.27 1.27)
+			)
+		)
+	)
 	(label "BOOT"
 		(at 110.49 92.71 0)
@@
 			)
 		)
-		(property "Datasheet" "https://wmsc.lcsc.com/wmsc/upload/file/pdf/v2/lcsc/2404260921_cjiang--Changjiang-Microelectronics-Tech-FXL0630-150-M_C177243.pdf"
+		(property "Datasheet" "https://wmsc.lcsc.com/wmsc/upload/file/pdf/v2/lcsc/1810201249_Murata-Electronics-LQM31PN2R2M00L_C171763.pdf"
 			(at 158.75 30.48 0)
 			(effects
@@
 			)
 		)
-		(property "Description" "3A 15uH Molding Choke ±20% 4.5A SMD,6.6x7mm Power Inductors ROHS "
+		(property "Description" "900mA 2.2uH ±20% 237.5mΩ 1206 Inductors (SMD) ROHS "
 			(at 158.75 30.48 0)
 			(effects
@@
 			)
 		)
-		(property "JLCPCB Part #" "C216156"
+		(property "JLCPCB Part #" "C171763"
 			(at 158.75 30.48 0)
 			(effects
@@
 			)
 		)
-		(property "Package" "L0805"
+		(property "Package" "1206"
 			(at 158.75 30.48 0)
 			(effects
@@
 					(unit 1)
 				)
+			)
+		)
+	)
+	(symbol
+		(lib_id "Connector:TestPoint")
+		(at 227.33 105.41 0)
+		(unit 1)
+		(exclude_from_sim no)
+		(in_bom yes)
+		(on_board yes)
+		(dnp no)
+		(fields_autoplaced yes)
+		(property "Reference" "TP5"
+			(at 229.87 100.8379 0)
+			(effects
+				(font
+					(size 1.27 1.27)
+				)
+				(justify left)
+			)
+		)
+		(property "Value" "3v3"
+			(at 229.87 103.3779 0)
+			(effects
+				(font
+					(size 1.27 1.27)
+				)
+				(justify left)
+			)
+		)
+		(property "Footprint" "TestPoint:TestPoint_THTPad_D1.0mm_Drill0.5mm"
+			(at 232.41 105.41 0)
+			(effects
+				(font
+					(size 1.27 1.27)
+				)
+				(hide yes)
+			)
+		)
+		(property "Datasheet" "~"
+			(at 232.41 105.41 0)
+			(effects
+				(font
+					(size 1.27 1.27)
+				)
+				(hide yes)
+			)
+		)
+		(property "Description" "test point"
+			(at 227.33 105.41 0)
+			(effects
+				(font
+					(size 1.27 1.27)
+				)
+				(hide yes)
+			)
+		)
+		(pin "1"
+		)
+		(instances
+			(project "Temperature_cluster"
+				(path "/c96faf72-0ed2-4ed1-a439-4e57053e11b5/65668258-1380-40f1-8f0c-18d3dfc5e1a1"
+					(reference "TP5")
+					(unit 1)
+				)

Commit message: Temp Cluster update
Parts:
- C14, C19: value 10v, 220uF -> 50v, 220uF; footprint Capacitor_SMD:CP_Elec_6.3x5.4 -> Capacitor_SMD:CP_Elec_10x10.5; JLCPCB Part # C72494 -> C365680; Package SMD,D6.3xL5.4mm -> SMD,D10xL10.5mm
Other:
- note added: "Input range 14V-32V"
- note removed: "Input range 14V-36V"
Changed lines of the file:
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@@
 		(title "Power Module")
 		(date "2024-06-28")
-		(rev "A")
+		(rev "B")
 		(company "D. Vaitiekus")
 		(comment 1 "AUGA Tech")
@@
 		)
 	)
-	(text "Input range\n14V-36V"
+	(text "Input range\n14V-32V"
 		(exclude_from_sim no)
 		(at 37.592 40.386 0)
@@
 			)
 		)
-		(property "Value" "10v, 220uF"
+		(property "Value" "50v, 220uF"
 			(at 131.064 47.498 90)
 			(effects
@@
 			)
 		)
-		(property "Footprint" "Capacitor_SMD:CP_Elec_6.3x5.4"
+		(property "Footprint" "Capacitor_SMD:CP_Elec_10x10.5"
 			(at 128.27 41.91 0)
 			(effects
@@
 			)
 		)
-		(property "Datasheet" "~"
+		(property "Datasheet" "https://wmsc.lcsc.com/wmsc/upload/file/pdf/v2/lcsc/1912111437_Rubycon-50TLV220MSPA10X10-5_C365680.pdf"
 			(at 128.27 41.91 0)
 			(effects
@@
 			)
 		)
-		(property "Description" "Polarized capacitor, small symbol"
+		(property "Description" "220uF 50V ±20% SMD,D10xL10.5mm  Aluminum Electrolytic Capacitors - SMD ROHS"
 			(at 128.27 41.91 0)
 			(effects
@@
 			)
 		)
-		(property "JLCPCB Part #" "C72494"
+		(property "JLCPCB Part #" "C365680"
 			(at 128.27 41.91 0)
 			(effects
@@
 			)
 		)
-		(property "Package" "SMD,D6.3xL5.4mm"
+		(property "Package" "SMD,D10xL10.5mm"
 			(at 128.27 41.91 0)
 			(effects
@@
 			)
 		)
-		(property "Value" "10v, 220uF"
+		(property "Value" "50v, 220uF"
 			(at 171.704 47.498 90)
 			(effects
@@
 			)
 		)
-		(property "Footprint" "Capacitor_SMD:CP_Elec_6.3x5.4"
+		(property "Footprint" "Capacitor_SMD:CP_Elec_10x10.5"
 			(at 168.91 41.91 0)
 			(effects
@@
 			)
 		)
-		(property "Datasheet" "~"
+		(property "Datasheet" "https://wmsc.lcsc.com/wmsc/upload/file/pdf/v2/lcsc/1912111437_Rubycon-50TLV220MSPA10X10-5_C365680.pdf"
 			(at 168.91 41.91 0)
 			(effects
@@
 			)
 		)
-		(property "Description" "Polarized capacitor, small symbol"
+		(property "Description" "220uF 50V ±20% SMD,D10xL10.5mm  Aluminum Electrolytic Capacitors - SMD ROHS"
 			(at 168.91 41.91 0)
 			(effects
@@
 			)
 		)
-		(property "JLCPCB Part #" "C72494"
+		(property "JLCPCB Part #" "C365680"
 			(at 168.91 41.91 0)
 			(effects
@@
 			)
 		)
-		(property "Package" "SMD,D6.3xL5.4mm"
+		(property "Package" "SMD,D10xL10.5mm"
 			(at 168.91 41.91 0)
 			(effects
