File: Temperature_cluster/Temperature_cluster.kicad_pcb (KiCad board)
At the start: 2 copper layers, 82.6 x 101.6 mm, 91 parts, among them J1 Header A, J2 DTM13-12PA-12PB, J3 Header B, U1 ESP32-DEVKITC-32D, U2 ADS1115IDGS - 1, U3 ADS1115IDGS - 1, U4 ADS1115IDGS - 2, U5 ADS1115IDGS - 2, U6 TPS5430DDAR, U7 AMS1117-3.3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

Commit message: PCB updates
Parts:
- removed U1: ESP32-DEVKITC-32D, 0_user_lib:MODULE_ESP32-DEVKITC-32D
- added J4: ESP32_Left, Connector_PinSocket_2.54mm:PinSocket_1x19_P2.54mm_Vertical, F.Cu at (177.0, 111.7)
- added J5: ESP32_Right, Connector_PinSocket_2.54mm:PinSocket_1x19_P2.54mm_Vertical, F.Cu at (151.6, 111.7)
- added J6: NTC_Internal, Connector_PinHeader_2.54mm:PinHeader_1x02_P2.54mm_Vertical, F.Cu at (160.5, 103.2)
- added J7: EXTRA1, Connector_PinHeader_2.54mm:PinHeader_1x10_P2.54mm_Vertical, F.Cu at (160.0, 54.6)
- added J8: EXTRA3, Connector_PinHeader_2.54mm:PinHeader_1x10_P2.54mm_Vertical, F.Cu at (160.0, 57.1)
- added J9: EXTRA2, Connector_PinHeader_2.54mm:PinHeader_1x10_P2.54mm_Vertical, F.Cu at (160.0, 59.7)
- added R28: 100k, Resistor_SMD:R_0805_2012Metric, F.Cu at (121.5, 116.1)
- added R29: 10K, Resistor_SMD:R_0805_2012Metric, F.Cu at (157.5, 103.2)
- added R30: 10K, Resistor_SMD:R_0805_2012Metric, F.Cu at (121.5, 112.6)
- added TP5: 3v3, TestPoint:TestPoint_THTPad_D1.0mm_Drill0.5mm, F.Cu at (127.5, 111.0)
- added TP6: CANH, TestPoint:TestPoint_THTPad_D1.0mm_Drill0.5mm, F.Cu at (160.0, 120.9)
- added TP7: CANL, TestPoint:TestPoint_THTPad_D1.0mm_Drill0.5mm, F.Cu at (156.0, 126.2)
- G1: moved to B.Cu
- J1: value Header A -> ESP32_Left
- J3: value Header B -> ESP32_Right
- U3: value ADS1115IDGS - 1 -> ADS1115IDGS - 3
- U5: value ADS1115IDGS - 2 -> ADS1115IDGS - 4
- moved G1 42.4 mm to (147.5, 124.7), turned to 180 degrees
Connections:
- J1 pad 11: /SCK -> /IO18
- J1 pad 12: /SO -> /IO19
- J1 pad 14: /INT -> /i2c_ADDR-4
- J1 pad 17: /IO22 -> /i2c_ADDR-3
- J1 pad 18: /SI -> /IO23
- J3 pad 12: /IO33 -> /NTC_INT
- J3 pad 13: /IO32 -> /VBAT_Sense
Routing:
- net /i2c_ADDR-3: track 81.2 -> 153.8 mm, vias 5 -> 6
- net /i2c_ADDR-4: track 77.5 -> 135.5 mm, vias 5 -> 6
- net /VBAT_Sense: track 0.00 -> 51.9 mm, vias 0 -> 1
- net /NTC_INT: track 0.00 -> 34.1 mm
- net +3.3VP: track 130.1 -> 148.0 mm
- net /IO33: track 7.60 -> 0.00 mm
- net /IO32: track 7.60 -> 0.00 mm
- net /SO: track 7.00 -> 0.00 mm
- net /SI: track 7.00 -> 0.00 mm
- net /SCK: track 7.00 -> 0.00 mm
- net /IO23: track 0.00 -> 7.00 mm
- net /IO22: track 7.00 -> 0.00 mm
- net /IO19: track 0.00 -> 7.00 mm
- net /IO18: track 0.00 -> 7.00 mm
- net /INT: track 7.00 -> 0.00 mm
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Other:
- board text added: "3v3"
- board text added: "5V"
- board text added: "60 Ohm"
- board text added: "ADS1115 - 1"
- board text added: "ADS1115 - 2"
- board text added: "ADS1115 - 3"
- board text added: "ADS1115 - 4"
- board text added: "BAT+"
- board text added: "BAT-"
- board text added: "CANH"
- board text added: "CANL"
- board text added: "D. Vaitiekus 2024-04-16 Temperature-Cluster Rev: A AUGA Tech"
- board text added: "ESP32-WROOM-32UE"
- board text added: "GND"
- board text added: "High side"
- board text added: "Low side"
- board text added: "NTC Pull Selectors"
- board text added: "NTC1"
- board text added: "NTC10"
- board text added: "NTC11"
- board text added: "NTC12"
- board text added: "NTC13"
- board text added: "NTC14"
- board text added: "NTC15"
- board text added: "NTC16"
- board text added: "NTC2"
- board text added: "NTC3"
- board text added: "NTC4"
- board text added: "NTC5"
- board text added: "NTC6"
- board text added: "NTC7"
- board text added: "NTC8"
- board text added: "NTC9"
- board text added: "NTCIN"
- board text added: "NTC_INT"
- board text added: "PU PD"
- board text added: "PWR_OK"

Commit message: Temp Cluster update
Parts:
- removed R3, R4, R5, R6: 5.1k, Resistor_SMD:R_0805_2012Metric
- added J10: Ext RGB connector, Connector_PinHeader_2.54mm:PinHeader_1x03_P2.54mm_Vertical, F.Cu at (132.0, 110.5)
- C14, C19: value 10v, 220uF -> 50v, 220uF; footprint Capacitor_SMD:CP_Elec_6.3x5.4 -> Capacitor_SMD:CP_Elec_10x10.5
- moved C21 11.5 mm to (129.8, 60.2), turned to -90 degrees
- moved C20 9.98 mm to (127.3, 60.2), turned to 90 degrees
- moved C15 9.26 mm to (123.6, 73.5), turned to -90 degrees
- moved TP5 7.74 mm to (123.8, 104.2)
- moved C19 5.90 mm to (119.4, 64.1), turned to -90 degrees
- moved C16 5.80 mm to (121.2, 73.5), turned to 90 degrees
- moved C14 3.37 mm to (118.4, 81.7), turned to -90 degrees
- moved L2 0.46 mm to (114.8, 73.2)
- moved D4 0.30 mm to (128.6, 71.5)
Connections:
- J3 pad 7: /ADC1-RDY -> /IO12
- J5 pad 7: /ADC1-RDY -> /IO12
Routing:
- net +3.3VP: track 148.0 -> 97.8 mm, vias 4 -> 2
- net /ADC1-RDY: track 45.5 -> 0.00 mm, vias 1 -> 0
- net /ADC3-RDY: track 8.54 -> 0.00 mm, vias 2 -> 0
- net /IO12: track 0.00 -> 7.60 mm
- net /ADC4-RDY: track 7.09 -> 0.00 mm, vias 2 -> 0
- net Vin_Filtered: track 32.4 -> 27.8 mm
- net /WS_LED: track 25.8 -> 30.2 mm
- net +5V: track 84.8 -> 88.5 mm
- net /ADC2-RDY: track 3.52 -> 0.00 mm
- net +3V3: track 56.4 -> 55.0 mm
- net GND: vias 139 -> 142
Other:
- board text added: "D. Vaitiekus 2024-08-02 Temperature-Cluster Rev: B AUGA Tech"
- board text removed: "D. Vaitiekus 2024-04-16 Temperature-Cluster Rev: A AUGA Tech"
