File: Temperature_cluster/Temperature_cluster.kicad_sch (KiCad schematic)
At the start: 41 parts, among them J2 DTM13-12PA-12PB, J2 Header A, J7 Header B, U1 ESP32-DEVKITC-32D, U2 ADS1115IDGS - 1, U3 ADS1115IDGS - 1, U4 ADS1115IDGS - 2, U5 ADS1115IDGS - 2

Commit message: PCB updates
Parts:
- added J4: ESP32_Left, Connector_PinSocket_2.54mm:PinSocket_1x19_P2.54mm_Vertical, symbol Connector_Generic:Conn_01x19
- added J5: ESP32_Right, Connector_PinSocket_2.54mm:PinSocket_1x19_P2.54mm_Vertical, symbol Connector_Generic:Conn_01x19
- added J6: NTC_Internal, Connector_PinHeader_2.54mm:PinHeader_1x02_P2.54mm_Vertical, symbol Connector:Conn_01x02_Pin
- added J7: EXTRA1, Connector_PinHeader_2.54mm:PinHeader_1x10_P2.54mm_Vertical, symbol Connector_Generic:Conn_01x10
- added J8: EXTRA3, Connector_PinHeader_2.54mm:PinHeader_1x10_P2.54mm_Vertical, symbol Connector_Generic:Conn_01x10
- added J9: EXTRA2, Connector_PinHeader_2.54mm:PinHeader_1x10_P2.54mm_Vertical, symbol Connector_Generic:Conn_01x10
- added R28: 100k, Resistor_SMD:R_0805_2012Metric, symbol Device:R_Small
- added R29, R30: 10K, Resistor_SMD:R_0805_2012Metric, symbol Device:R_Small
- J2: value Header A -> ESP32_Left; JLCPCB Part # C22373905 -> C319202; now not fitted
- J7: value Header B -> ESP32_Right; JLCPCB Part # C22373905 -> C319202; now not fitted
- U1: now not fitted; now left out of the parts list
- U3: value ADS1115IDGS - 1 -> ADS1115IDGS - 3
- U5: value ADS1115IDGS - 2 -> ADS1115IDGS - 4
Connections:
- net +3.3VP: now also J5.19 (Pin_19), J6.2 (Pin_2); no longer U1.J2-1 (3V3)
- net +5V: now also J5.1 (Pin_1); no longer U1.J2-19 (EXT_5V)
- net ADC1-RDY: now also J5.7 (Pin_7); no longer U1.J2-13 (IO12)
- net CAN_RX: now also J4.7 (Pin_7); no longer U1.J3-13 (IO4)
- net CAN_S: now also J4.5 (Pin_5); no longer U1.J3-15 (IO2)
- net CAN_TX: now also J4.10 (Pin_10); no longer U1.J3-10 (IO5)
- net CLK: now also J4.1 (Pin_1); no longer U1.J3-19 (CLK)
- net CMD: now also J5.2 (Pin_2); no longer U1.J2-18 (CMD)
- net EN: now also J5.18 (Pin_18); no longer U1.J2-2 (EN)
- net GND: now also J4.13 (Pin_13), J4.19 (Pin_19), J5.6 (Pin_6), R29.2, R30.1; no longer U1.J2-14 (GND1), U1.J3-1 (GND3), U1.J3-7 (GND2)
- net IO0: now also J4.6 (Pin_6); no longer U1.J3-14 (IO0)
- net IO14: now also J5.8 (Pin_8); no longer U1.J2-12 (IO14)
- net IO15: now also J4.4 (Pin_4); no longer U1.J3-16 (IO15)
- net IO16: now also J4.8 (Pin_8); no longer U1.J3-12 (IO16)
- net IO17: now also J4.9 (Pin_9); no longer U1.J3-11 (IO17)
- net IO18: now also J4.11 (Pin_11); no longer U1.J3-9 (IO18)
- net IO19: now also J4.12 (Pin_12); no longer U1.J3-8 (IO19)
- net IO23: now also J4.18 (Pin_18); no longer U1.J3-2 (IO23)
- net IO25: now also J5.11 (Pin_11); no longer U1.J2-9 (IO25)
- net IO26: now also J5.10 (Pin_10); no longer U1.J2-10 (IO26)
- net IO27: now also J5.9 (Pin_9); no longer U1.J2-11 (IO27)
- net IO34: now also J5.15 (Pin_15); no longer U1.J2-5 (IO34)
- net IO35: now also J5.14 (Pin_14); no longer U1.J2-6 (IO35)
- net RXD0: now also J4.15 (Pin_15); no longer U1.J3-5 (RXD0)
- net SD0: now also J4.2 (Pin_2); no longer U1.J3-18 (SD0)
- net SD1: now also J4.3 (Pin_3); no longer U1.J3-17 (SD1)
- net SD2: now also J5.4 (Pin_4); no longer U1.J2-16 (SD2)
- net SD3: now also J5.3 (Pin_3); no longer U1.J2-17 (SD3)
- net TXD0: now also J4.16 (Pin_16); no longer U1.J3-4 (TXD0)
- net VBat+: now also R28.1
- net VN: now also J5.16 (Pin_16); no longer U1.J2-4 (SENSOR_VN)
- net VP: now also J5.17 (Pin_17); no longer U1.J2-3 (SENSOR_VP)
- net WS_LED: now also J5.5 (Pin_5); no longer U1.J2-15 (IO13)
- net i2c_ADDR-3: now also J4.17 (Pin_17); no longer U1.J3-3 (IO22)
- net i2c_ADDR-4: now also J4.14 (Pin_14); no longer U1.J3-6 (IO21)
- net IO32: no longer names the net of U1.J2-7 (IO32)
- net IO32: no longer J7.13 (Pin_13)
- net IO33: no longer names the net of U1.J2-8 (IO33)
- net IO33: no longer J7.12 (Pin_12)
- new net: J7.1 (Pin_1), J8.1 (Pin_1), J9.1 (Pin_1)
- new net: J7.10 (Pin_10), J8.10 (Pin_10), J9.10 (Pin_10)
- new net: J7.2 (Pin_2), J8.2 (Pin_2), J9.2 (Pin_2)
- new net: J7.3 (Pin_3), J8.3 (Pin_3), J9.3 (Pin_3)
- new net: J7.4 (Pin_4), J8.4 (Pin_4), J9.4 (Pin_4)
- new net: J7.5 (Pin_5), J8.5 (Pin_5), J9.5 (Pin_5)
- new net: J7.6 (Pin_6), J8.6 (Pin_6), J9.6 (Pin_6)
- new net: J7.7 (Pin_7), J8.7 (Pin_7), J9.7 (Pin_7)
- new net: J7.8 (Pin_8), J8.8 (Pin_8), J9.8 (Pin_8)
- new net: J7.9 (Pin_9), J8.9 (Pin_9), J9.9 (Pin_9)
- new net NTC_INT: J5.12 (Pin_12), J6.1 (Pin_1), J7.12 (Pin_12), R29.1
- new net VBAT_Sense: J5.13 (Pin_13), J7.13 (Pin_13), R28.2, R30.2
Other:
- note added: "36V -> 3.6V 14V -> 1.4V 12V -> 1.2V 10V -> 1.0V"
- note added: "ADC1 Address: 1001000 0x48"
- note added: "ADC2 Address: 1001001 0x49"
- note added: "ADC3 Address: 1001010 0x4A"
- note added: "ADC4 Address: 1001011 0x4B"
- note added: "Battery Voltage monitor"
- note added: "Input range: 14-36V"
- note added: "NTC internal probe solder points"
- note added: "You should only use GPIO-12 as an output pin. Or at least it should never be pulled up or down by something external. The state of this pin will determine the flash voltage. If you have a board which needs the lower voltage of both options, you will fry the chip. For the other option, it will just "not work""
- note removed: "ADC1 Address: 1001000"
- note removed: "ADC2 Address: 1001001"
- note removed: "ADC3 Address: 1001010"
- note removed: "ADC4 Address: 1001011"
- company: (none) -> D. Vaitiekus
- title: (none) -> Temp Cluster
- moved on the sheet: C1

Commit message: Temp Cluster update
Parts:
- removed R3, R4, R5, R6: 5.1k, Resistor_SMD:R_0805_2012Metric, symbol Device:R_Small
- added J10: Ext RGB connector, Connector_PinHeader_2.54mm:PinHeader_1x03_P2.54mm_Vertical, symbol Connector_Generic:Conn_01x03
Connections:
- net +5V: now also J10.1 (Pin_1)
- net ADC1-RDY: no longer J5.7 (Pin_7), J7.7 (Pin_7)
- net GND: now also J10.3 (Pin_3)
- net WS_LED: now also J10.2 (Pin_2)
- new net IO12: J5.7 (Pin_7), J7.7 (Pin_7)
- no-connect marks 1 -> 5
Other:
- note added: "32V -> 3.2V 14V -> 1.4V 12V -> 1.2V 10V -> 1.0V"
- note added: "Input range: 14-32V"
- note removed: "36V -> 3.6V 14V -> 1.4V 12V -> 1.2V 10V -> 1.0V"
- note removed: "Input range: 14-36V"
- note removed: "You should only use GPIO-12 as an output pin. Or at least it should never be pulled up or down by something external. The state of this pin will determine the flash voltage. If you have a board which needs the lower voltage of both options, you will fry the chip. For the other option, it will just "not work""
